File: AVR-USB2SERIAL.sch (EAGLE design)
At the start: 0 parts

Commit message: Micro-controller connections
Parts:
- added C1, C2, C3, C4, C5, C6: 100nF, rcl:C-EUC0805
- added LED1, LED2: (no value), led:LEDCHIPLED_0805
- added MICRO_USB: 10118192-0001LF, 10118192-0001LF:10118192-0001LF
- added R1: 10K, rcl:R-EU_R0805
- added R2, R3: 1K, rcl:R-EU_R0805
- added U1: FTDI_FT232RL-REELFTDI_FT232RL-REEL_0_0, FTDI - FT232RL-Reel:FTDI_FT232RL-REELFTDI_FT232RL-REEL_0_0
- added U2: MICROCHIP_-_ATMEL_ATMEGA328-AUMICROCHIP_-_ATMEL_ATMEGA328-A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, Atmel - ATMEGA328-AU:MICROCHIP_-_ATMEL_ATMEGA328-AUMICROCHIP_-_ATMEL_ATMEGA328-AU_0_0
Connections:
- new net +3V3: C1.2, U1.3V3OUT
- new net +5V: C2.1, C3.1, C4.2, C5.2, C6.1, MICRO_USB.VUSB, R1.1, R2.2, R3.2, U1.VCC, U1.VCCIO, U2.1_VCC, U2.2_VCC, U2.AVCC
- new net GND: C1.1, C2.2, C3.2, C4.1, C5.1, C6.2, MICRO_USB.GND, MICRO_USB.ID, MICRO_USB.SHIELD, U1.1_GND, U1.2_GND, U1.3_GND, U1.AGND, U2.1_GND, U2.2_GND, U2.3_GND
- new net N$1: LED1.C, U1.CBUS0
- new net N$2: R1.2, U1.!RESET!
- new net N$3: LED1.A, R2.1
- new net N$4: LED2.A, R3.1
- new net N$5: LED2.C, U1.CBUS1
- new net RXD: U1.RXD, U2.!PD1!(TXD/PCINT17)
- new net TXD: U1.TXD, U2.!PD0!(RXD/PCINT16)
- new net USB_DM: MICRO_USB.D-, U1.USBDM
- new net USB_DP: MICRO_USB.D+, U1.USBDP

Commit message: completed common connections
Parts:
- added C7, C8: 100nF, rcl:C-EUC0805
- added LED3, LED4: (no value), led:LEDCHIPLED_0805
- added P1: M-1X03-SIP-100-32, con-headers-jp:M-1X03-SIP-100-32
- added Q1: (no value), crystal:CRYSTALHC49UP
- added R4: 1K, rcl:R-EU_R0805
- added SW1: TE_CONNECTIVITY_ALCOSWITCH_FSM6JSMATE_CONNECTIVITY_ALCOSWIT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, TE Connectivity Alcoswitch - FSM6JSMA:TE_CONNECTIVITY_ALCOSWITCH_FSM6JSMATE_CONNECTIVITY_ALCOSWITCH_FSM6JSMA_0_0
Connections:
- new net AREF: P1.2, U2.AREF
- new net N$6: C7.1, Q1.2, U2.!PB6!(PCINT6/XTAL1/TOSC1)
- new net N$7: C8.1, Q1.1, U2.!PB7!(PCINT7/XTAL2/TOSC2)
- new net N$8: LED4.C, R4.2
- new net RESET: SW1.1, U2.!RESET!/PCINT14)
- net +3V3: now also P1.3
- net +5V: now also LED4.A, P1.1
- net GND: now also C7.2, C8.2, R4.1, SW1.3
- net N$1: now also LED3.C
- net N$3: now also LED3.A
Changed lines of the file:
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@@
 <part name="GND11" library="supply1" library_urn="urn:adsk.eagle:library:371" deviceset="GND" device=""/>
 <part name="GND12" library="supply1" library_urn="urn:adsk.eagle:library:371" deviceset="GND" device=""/>
+<part name="Q1" library="crystal" library_urn="urn:adsk.eagle:library:204" deviceset="CRYSTAL" device="HC49UP" package3d_urn="urn:adsk.eagle:package:12078/1"/>
+<part name="C7" library="rcl" library_urn="urn:adsk.eagle:library:334" deviceset="C-EU" device="C0805" package3d_urn="urn:adsk.eagle:package:23617/2" value="100nF"/>
+<part name="C8" library="rcl" library_urn="urn:adsk.eagle:library:334" deviceset="C-EU" device="C0805" package3d_urn="urn:adsk.eagle:package:23617/2" value="100nF"/>
+<part name="GND13" library="supply1" library_urn="urn:adsk.eagle:library:371" deviceset="GND" device=""/>
+<part name="P1" library="con-headers-jp" deviceset="M-1X03-" device="SIP-100-32"/>
+<part name="+3V2" library="supply1" library_urn="urn:adsk.eagle:library:371" deviceset="+3V3" device=""/>
+<part name="P+6" library="supply1" library_urn="urn:adsk.eagle:library:371" deviceset="+5V" device=""/>
+<part name="R4" library="rcl" library_urn="urn:adsk.eagle:library:334" deviceset="R-EU_" device="R0805" package3d_urn="urn:adsk.eagle:package:23553/2" value="1K"/>
+<part name="LED3" library="led" library_urn="urn:adsk.eagle:library:259" deviceset="LED" device="CHIPLED_0805" package3d_urn="urn:adsk.eagle:package:15821/2"/>
+<part name="LED4" library="led" library_urn="urn:adsk.eagle:library:259" deviceset="LED" device="CHIPLED_0805" package3d_urn="urn:adsk.eagle:package:15821/2"/>
+<part name="GND14" library="supply1" library_urn="urn:adsk.eagle:library:371" deviceset="GND" device=""/>
+<part name="SW1" library="TE Connectivity Alcoswitch - FSM6JSMA" deviceset="TE_CONNECTIVITY_ALCOSWITCH_FSM6JSMA" device="TE_CONNECTIVITY_ALCOSWITCH_FSM6JSMA_0_0"/>
+<part name="GND15" library="supply1" library_urn="urn:adsk.eagle:library:371" deviceset="GND" device=""/>
 </parts>
 <sheets>
@@
 <instance part="GND12" gate="1" x="165.1" y="2.54" smashed="yes">
 <attribute name="VALUE" x="162.56" y="0" size="1.778" layer="96"/>
+</instance>
+<instance part="Q1" gate="G$1" x="231.14" y="10.16" smashed="yes" rot="R90">
+<attribute name="NAME" x="235.204" y="7.62" size="1.778" layer="95" rot="R90"/>
+<attribute name="VALUE" x="233.68" y="12.7" size="1.778" layer="96" rot="R90"/>
+</instance>
+<instance part="C7" gate="G$1" x="238.76" y="15.24" smashed="yes" rot="R90">
+<attribute name="NAME" x="238.379" y="16.764" size="1.778" layer="95" rot="R90"/>
+<attribute name="VALUE" x="243.459" y="16.764" size="1.778" layer="96" rot="R90"/>
+</instance>
+<instance part="C8" gate="G$1" x="241.3" y="5.08" smashed="yes" rot="R90">
+<attribute name="NAME" x="240.919" y="6.604" size="1.778" layer="95" rot="R90"/>
+<attribute name="VALUE" x="245.999" y="6.604" size="1.778" layer="96" rot="R90"/>
+</instance>
+<instance part="GND13" gate="1" x="254" y="5.08" smashed="yes">
+<attribute name="VALUE" x="251.46" y="2.54" size="1.778" layer="96"/>
+</instance>
+<instance part="P1" gate="G$1" x="162.56" y="50.8" smashed="yes">
+<attribute name="VALUE" x="161.29" y="43.18" size="1.778" layer="96"/>
+<attribute name="NAME" x="161.29" y="56.642" size="1.778" layer="95"/>
+</instance>
+<instance part="+3V2" gate="G$1" x="142.24" y="50.8" smashed="yes">
+<attribute name="VALUE" x="139.7" y="45.72" size="1.778" layer="96" rot="R90"/>
+</instance>
+<instance part="P+6" gate="1" x="142.24" y="58.42" smashed="yes">
+<attribute name="VALUE" x="139.7" y="53.34" size="1.778" layer="96" rot="R90"/>
+</instance>
+<instance part="R4" gate="G$1" x="144.78" y="93.98" smashed="yes">
+<attribute name="NAME" x="140.97" y="95.4786" size="1.778" layer="95"/>
+<attribute name="VALUE" x="140.97" y="90.678" size="1.778" layer="96"/>
+</instance>
+<instance part="LED3" gate="G$1" x="129.54" y="38.1" smashed="yes" rot="R270">
+<attribute name="NAME" x="124.968" y="34.544" size="1.778" layer="95"/>
+<attribute name="VALUE" x="124.968" y="32.385" size="1.778" layer="96"/>
+</instance>
+<instance part="LED4" gate="G$1" x="157.48" y="91.44" smashed="yes" rot="R270">
+<attribute name="NAME" x="152.908" y="87.884" size="1.778" layer="95"/>
+<attribute name="VALUE" x="152.908" y="85.725" size="1.778" layer="96"/>
+</instance>
+<instance part="GND14" gate="1" x="129.54" y="86.36" smashed="yes">
+<attribute name="VALUE" x="127" y="83.82" size="1.778" layer="96"/>
+</instance>
+<instance part="SW1" gate="G$0" x="203.2" y="111.76" smashed="yes">
+<attribute name="NAME" x="203.2" y="109.22" size="2.54" layer="95" align="top-left"/>
+</instance>
+<instance part="GND15" gate="1" x="185.42" y="91.44" smashed="yes">
+<attribute name="VALUE" x="182.88" y="88.9" size="1.778" layer="96"/>
 </instance>
 </instances>
@@
 <wire x1="167.64" y1="71.12" x2="167.64" y2="76.2" width="0.1524" layer="91"/>
 <junction x="167.64" y="76.2"/>
+<pinref part="LED4" gate="G$1" pin="A"/>
+<wire x1="160.02" y1="91.44" x2="160.02" y2="83.82" width="0.1524" layer="91"/>
+<wire x1="160.02" y1="83.82" x2="157.48" y2="83.82" width="0.1524" layer="91"/>
+<wire x1="157.48" y1="83.82" x2="157.48" y2="81.28" width="0.1524" layer="91"/>
+<junction x="157.48" y="81.28"/>
+</segment>
+<segment>
+<pinref part="P1" gate="G$1" pin="1"/>
+<pinref part="P+6" gate="1" pin="+5V"/>
+<wire x1="142.24" y1="55.88" x2="142.24" y2="53.34" width="0.1524" layer="91"/>
+<wire x1="142.24" y1="53.34" x2="157.48" y2="53.34" width="0.1524" layer="91"/>
 </segment>
 </net>
@@
 <junction x="167.64" y="10.16"/>
 </segment>
+<segment>
+<pinref part="C7" gate="G$1" pin="2"/>
+<wire x1="243.84" y1="15.24" x2="254" y2="15.24" width="0.1524" layer="91"/>
+<pinref part="GND13" gate="1" pin="GND"/>
+<wire x1="254" y1="15.24" x2="254" y2="10.16" width="0.1524" layer="91"/>
+<pinref part="C8" gate="G$1" pin="2"/>
+<wire x1="254" y1="10.16" x2="254" y2="7.62" width="0.1524" layer="91"/>
+<wire x1="246.38" y1="5.08" x2="248.92" y2="5.08" width="0.1524" layer="91"/>
+<wire x1="248.92" y1="5.08" x2="248.92" y2="10.16" width="0.1524" layer="91"/>
+<wire x1="248.92" y1="10.16" x2="254" y2="10.16" width="0.1524" layer="91"/>
+<junction x="254" y="10.16"/>
+</segment>
+<segment>
+<pinref part="GND14" gate="1" pin="GND"/>
+<wire x1="129.54" y1="88.9" x2="129.54" y2="93.98" width="0.1524" layer="91"/>
+<pinref part="R4" gate="G$1" pin="1"/>
+<wire x1="129.54" y1="93.98" x2="139.7" y2="93.98" width="0.1524" layer="91"/>
+</segment>
+<segment>
+<pinref part="SW1" gate="G$0" pin="3"/>
+<wire x1="198.12" y1="96.52" x2="185.42" y2="96.52" width="0.1524" layer="91"/>
+<pinref part="GND15" gate="1" pin="GND"/>
+<wire x1="185.42" y1="96.52" x2="185.42" y2="93.98" width="0.1524" layer="91"/>
+</segment>
 </net>
 <net name="USB_DM" class="0">
@@
 <junction x="66.04" y="60.96"/>
 </segment>
+<segment>
+<pinref part="P1" gate="G$1" pin="3"/>
+<pinref part="+3V2" gate="G$1" pin="+3V3"/>
+<wire x1="142.24" y1="48.26" x2="157.48" y2="48.26" width="0.1524" layer="91"/>
+</segment>
 </net>
 <net name="N$2" class="0">
@@
 <pinref part="LED1" gate="G$1" pin="C"/>
 <wire x1="116.84" y1="38.1" x2="124.46" y2="38.1" width="0.1524" layer="91"/>
+<pinref part="LED3" gate="G$1" pin="C"/>
+<junction x="124.46" y="38.1"/>
 </segment>
 </net>
@@
 <pinref part="R2" gate="G$1" pin="1"/>
 <wire x1="132.08" y1="38.1" x2="134.62" y2="38.1" width="0.1524" layer="91"/>
+<pinref part="LED3" gate="G$1" pin="A"/>
+<junction x="132.08" y="38.1"/>
 </segment>
 </net>
@@
 </segment>
 </net>
+<net name="RESET" class="0">
+<segment>
+<pinref part="U2" gate="G$0" pin="!RESET!/PCINT14)"/>
+<wire x1="226.06" y1="55.88" x2="233.68" y2="55.88" width="0.1524" layer="91"/>
+<label x="231.14" y="55.88" size="1.778" layer="95"/>
+</segment>
+<segment>
+<pinref part="SW1" gate="G$0" pin="1"/>
+<wire x1="198.12" y1="104.14" x2="185.42" y2="104.14" width="0.1524" layer="91"/>
+<label x="185.42" y="104.14" size="1.778" layer="95"/>
+</segment>
+</net>
+<net name="N$6" class="0">
+<segment>
+<pinref part="U2" gate="G$0" pin="!PB6!(PCINT6/XTAL1/TOSC1)"/>
+<pinref part="Q1" gate="G$1" pin="2"/>
+<wire x1="226.06" y1="12.7" x2="231.14" y2="12.7" width="0.1524" layer="91"/>
+<pinref part="C7" gate="G$1" pin="1"/>
+<wire x1="231.14" y1="12.7" x2="236.22" y2="12.7" width="0.1524" layer="91"/>
+<wire x1="236.22" y1="12.7" x2="236.22" y2="15.24" width="0.1524" layer="91"/>
+<junction x="231.14" y="12.7"/>
+</segment>
+</net>
+<net name="N$7" class="0">
+<segment>
+<pinref part="U2" gate="G$0" pin="!PB7!(PCINT7/XTAL2/TOSC2)"/>
+<wire x1="226.06" y1="10.16" x2="226.06" y2="7.62" width="0.1524" layer="91"/>
+<pinref part="Q1" gate="G$1" pin="1"/>
+<wire x1="226.06" y1="7.62" x2="231.14" y2="7.62" width="0.1524" layer="91"/>
+<pinref part="C8" gate="G$1" pin="1"/>
+<wire x1="231.14" y1="7.62" x2="231.14" y2="5.08" width="0.1524" layer="91"/>
+<wire x1="231.14" y1="5.08" x2="238.76" y2="5.08" width="0.1524" layer="91"/>
+<junction x="231.14" y="7.62"/>
+</segment>
+</net>
+<net name="AREF" class="0">
+<segment>
+<pinref part="U2" gate="G$0" pin="AREF"/>
+<wire x1="175.26" y1="66.04" x2="165.1" y2="66.04" width="0.1524" layer="91"/>
+<label x="165.1" y="66.04" size="1.778" layer="95"/>
+</segment>
+<segment>
+<pinref part="P1" gate="G$1" pin="2"/>
+<wire x1="157.48" y1="50.8" x2="149.86" y2="50.8" width="0.1524" layer="91"/>
+<label x="149.86" y="50.8" size="1.778" layer="95"/>
+</segment>
+</net>
+<net name="N$8" class="0">
+<segment>
+<pinref part="R4" gate="G$1" pin="2"/>
+<pinref part="LED4" gate="G$1" pin="C"/>
+<wire x1="149.86" y1="93.98" x2="149.86" y2="91.44" width="0.1524" layer="91"/>
+<wire x1="149.86" y1="91.44" x2="152.4" y2="91.44" width="0.1524" layer="91"/>
+</segment>
+</net>

Commit message: unrouted board
Parts:
- removed LED3: (no value), led:LEDCHIPLED_0805
- added RX, TX: TPB1,27, testpad:TPB1,27
Connections:
- net N$1: now also LED1.A, R2.1; no longer LED1.C, LED3.C, U1.CBUS0
- net N$3: now also LED1.C, U1.CBUS0; no longer LED1.A, LED3.A, R2.1
- net RXD: now also RX.TP
- net TXD: now also TX.TP
Changed lines of the file:
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@@
 </variantdefs>
 <classes>
-<class number="0" name="default" width="0" drill="0">
+<class number="0" name="default" width="0.5" drill="0.3">
+<clearance class="0" value="0.3"/>
+</class>
+<class number="1" name="POWER" width="0.8" drill="0.3">
+<clearance class="1" value="0.3"/>
 </class>
 </classes>
@@
 <part name="P+6" library="supply1" library_urn="urn:adsk.eagle:library:371" deviceset="+5V" device=""/>
 <part name="R4" library="rcl" library_urn="urn:adsk.eagle:library:334" deviceset="R-EU_" device="R0805" package3d_urn="urn:adsk.eagle:package:23553/2" value="1K"/>
-<part name="LED3" library="led" library_urn="urn:adsk.eagle:library:259" deviceset="LED" device="CHIPLED_0805" package3d_urn="urn:adsk.eagle:package:15821/2"/>
 <part name="LED4" library="led" library_urn="urn:adsk.eagle:library:259" deviceset="LED" device="CHIPLED_0805" package3d_urn="urn:adsk.eagle:package:15821/2"/>
 <part name="GND14" library="supply1" library_urn="urn:adsk.eagle:library:371" deviceset="GND" device=""/>
 <part name="SW1" library="TE Connectivity Alcoswitch - FSM6JSMA" deviceset="TE_CONNECTIVITY_ALCOSWITCH_FSM6JSMA" device="TE_CONNECTIVITY_ALCOSWITCH_FSM6JSMA_0_0"/>
 <part name="GND15" library="supply1" library_urn="urn:adsk.eagle:library:371" deviceset="GND" device=""/>
+<part name="RX" library="testpad" library_urn="urn:adsk.eagle:library:385" deviceset="TP" device="B1,27" package3d_urn="urn:adsk.eagle:package:27944/2"/>
+<part name="TX" library="testpad" library_urn="urn:adsk.eagle:library:385" deviceset="TP" device="B1,27" package3d_urn="urn:adsk.eagle:package:27944/2"/>
 </parts>
 <sheets>
@@
 <attribute name="VALUE" x="140.97" y="90.678" size="1.778" layer="96"/>
 </instance>
-<instance part="LED3" gate="G$1" x="129.54" y="38.1" smashed="yes" rot="R270">
-<attribute name="NAME" x="124.968" y="34.544" size="1.778" layer="95"/>
-<attribute name="VALUE" x="124.968" y="32.385" size="1.778" layer="96"/>
-</instance>
 <instance part="LED4" gate="G$1" x="157.48" y="91.44" smashed="yes" rot="R270">
 <attribute name="NAME" x="152.908" y="87.884" size="1.778" layer="95"/>
@@
 <instance part="GND15" gate="1" x="185.42" y="91.44" smashed="yes">
 <attribute name="VALUE" x="182.88" y="88.9" size="1.778" layer="96"/>
+</instance>
+<instance part="RX" gate="G$1" x="248.92" y="53.34" smashed="yes" rot="R270">
+<attribute name="NAME" x="250.19" y="54.61" size="1.778" layer="95" rot="R270"/>
+<attribute name="TP_SIGNAL_NAME" x="247.65" y="52.07" size="1.778" layer="97" rot="R270"/>
+</instance>
+<instance part="TX" gate="G$1" x="248.92" y="48.26" smashed="yes" rot="R270">
+<attribute name="NAME" x="250.19" y="49.53" size="1.778" layer="95" rot="R270"/>
+<attribute name="TP_SIGNAL_NAME" x="247.65" y="46.99" size="1.778" layer="97" rot="R270"/>
 </instance>
 </instances>
@@
 </busses>
 <nets>
-<net name="+5V" class="0">
+<net name="+5V" class="1">
 <segment>
 <pinref part="P+1" gate="1" pin="+5V"/>
@@
 </segment>
 </net>
-<net name="GND" class="0">
+<net name="GND" class="1">
 <segment>
 <pinref part="GND1" gate="1" pin="GND"/>
@@
 </segment>
 </net>
-<net name="+3V3" class="0">
+<net name="+3V3" class="1">
 <segment>
 <pinref part="+3V1" gate="G$1" pin="+3V3"/>
@@
 </segment>
 </net>
-<net name="N$1" class="0">
-<segment>
-<pinref part="U1" gate="G$0" pin="CBUS0"/>
-<pinref part="LED1" gate="G$1" pin="C"/>
-<wire x1="116.84" y1="38.1" x2="124.46" y2="38.1" width="0.1524" layer="91"/>
-<pinref part="LED3" gate="G$1" pin="C"/>
-<junction x="124.46" y="38.1"/>
-</segment>
-</net>
-<net name="N$3" class="0">
-<segment>
-<pinref part="LED1" gate="G$1" pin="A"/>
-<pinref part="R2" gate="G$1" pin="1"/>
-<wire x1="132.08" y1="38.1" x2="134.62" y2="38.1" width="0.1524" layer="91"/>
-<pinref part="LED3" gate="G$1" pin="A"/>
-<junction x="132.08" y="38.1"/>
-</segment>
-</net>
 <net name="N$4" class="0">
 <segment>
@@
 <label x="231.14" y="50.8" size="1.778" layer="95"/>
 </segment>
+<segment>
+<pinref part="TX" gate="G$1" pin="TP"/>
+<wire x1="246.38" y1="48.26" x2="241.3" y2="48.26" width="0.1524" layer="91"/>
+<label x="241.3" y="48.26" size="1.778" layer="95"/>
+</segment>
 </net>
 <net name="RXD" class="0">
@@
 <wire x1="226.06" y1="48.26" x2="233.68" y2="48.26" width="0.1524" layer="91"/>
 <label x="231.14" y="48.26" size="1.778" layer="95"/>
+</segment>
+<segment>
+<pinref part="RX" gate="G$1" pin="TP"/>
+<wire x1="246.38" y1="53.34" x2="241.3" y2="53.34" width="0.1524" layer="91"/>
+<label x="241.3" y="53.34" size="1.778" layer="95"/>
 </segment>
 </net>
@@
 </segment>
 </net>
+<net name="N$1" class="0">
+<segment>
+<pinref part="R2" gate="G$1" pin="1"/>
+<pinref part="LED1" gate="G$1" pin="A"/>
+<wire x1="134.62" y1="38.1" x2="132.08" y2="38.1" width="0.1524" layer="91"/>
+</segment>
+</net>
+<net name="N$3" class="0">
+<segment>
+<pinref part="LED1" gate="G$1" pin="C"/>
+<pinref part="U1" gate="G$0" pin="CBUS0"/>
+<wire x1="124.46" y1="38.1" x2="116.84" y2="38.1" width="0.1524" layer="91"/>
+</segment>
+</net>
